File: games/idle/hardware/esp32-idle-game.kicad_pcb (KiCad board)
At the start: 2 copper layers, 62 x 100 mm, 17 parts, among them J1 ILI9341 2.8in, J2 ESP32 DevKit V1, J3 ESP32 DevKit V1, Q1 S8050 (EBC), SW1 6x6 tact, SW2 6x6 tact, SW3 6x6 tact, SW4 6x6 tact, SW5 6x6 tact

Commit message: feat: ajustes design hardware
Parts:
- BZ1: value Passive buzzer 9mm -> Passive buzzer 12mm; footprint Buzzer_D9mm_P4mm -> Buzzer_D12mm_P6.5-7.6mm
- moved J1 33.0 mm to (14.5, 66.3), turned to 90 degrees
Routing:
- net TFT_CS: track 80.5 -> 62.0 mm
- net TFT_MOSI: track 62.4 -> 45.5 mm
- net GND: track 170.7 -> 186.1 mm
- net EN: track 34.8 -> 49.0 mm, vias 0 -> 1
- net TFT_DC: track 74.1 -> 62.0 mm, vias 1 -> 0
- net BTN_BACK: track 68.5 -> 79.4 mm
- net TFT_MISO: track 37.7 -> 46.2 mm, vias 0 -> 1
- net +5V: track 85.8 -> 80.8 mm
- net BTN_UP: track 76.9 -> 72.0 mm
- net TFT_LED: track 60.3 -> 64.6 mm
- net TFT_SCK: track 40.0 -> 37.7 mm, vias 1 -> 0
- net BUZ_N: track 26.0 -> 24.3 mm
- net BTN_MENU: track 83.7 -> 82.6 mm
- net BTN_CONFIRM: track 60.4 -> 61.3 mm
Other:
- board text added: "v5.1"
- board text removed: "v5.0"
