File: games/idle/hardware/esp32-idle-game.kicad_pcb (KiCad board)
At the start: 2 copper layers, 62 x 100 mm, 17 parts, among them J1 ILI9341 2.8in, J2 ESP32 DevKit V1, J3 ESP32 DevKit V1, Q1 S8050 (EBC), SW1 6x6 tact, SW2 6x6 tact, SW3 6x6 tact, SW4 6x6 tact, SW5 6x6 tact

Commit message: refactor(hardware): rename menu/back buttons to right/left
The D-pad's side buttons step through the screens, so the nets and
silkscreen now say BTN_RIGHT/BTN_LEFT and RIGHT/LEFT. Board regenerated
and re-routed; DRC clean.

Co-Authored-By: Claude Opus 5.5 <noreply@anthropic.com>
Connections:
- net BTN_BACK renamed BTN_LEFT
- net BTN_MENU renamed BTN_RIGHT
Other:
- board text added: "LEFT"
- board text added: "RIGHT"
- board text removed: "BACK"
- board text removed: "MENU"
